File: Hardware/EET_BMS_Layout/eet_bms Rev. 1.kicad_sch (KiCad schematic)
At the start: 4 parts

Commit message: fixed a bug in the firmware. Added in Hardware documentation
Other:
- sheet Current Sense Amplifier renamed Bidirectional Switch and Current Sense Amplifier
